Commit message: 准备把机械臂的名字改回來,方便后续与实体整合

File: my_jaka_zu5_moveit_config/config/jaka_robot.ros2_control.xacro (robot description, xacro)
@@ -1,10 +1,15 @@
 <?xml version="1.0"?>
 <robot xmlns:xacro="http://www.ros.org/wiki/xacro">
-    <xacro:macro name="jaka_robot_ros2_control" params="name initial_positions_file">
-        <xacro:property name="initial_positions" value="${load_yaml(initial_positions_file)['initial_positions']}"/>
+    <xacro:macro name="jaka_robot_ros2_control" params="name initial_positions_file use_gazebo use_rviz_sim">
+        <xacro:property name="initial_positions" value="${xacro.load_yaml(initial_positions_file)['initial_positions']}"/>
         <ros2_control name="${name}" type="system">
             <hardware>
-                <!-- By default, set up controllers for simulation. This won't work on real hardware -->
-                <plugin>mock_components/GenericSystem</plugin>
+              <xacro:if value="${use_gazebo}">
+                  <!-- <plugin>gazebo_ros2_control/GazeboSystem</plugin> -->
+                  <plugin>ign_ros2_control/IgnitionSystem</plugin>
+              </xacro:if>
+              <xacro:if value="${use_rviz_sim}">
+                  <plugin>mock_components/GenericSystem</plugin>
+              </xacro:if>
             </hardware>
             <joint name="joint_1">

File: my_jaka_zu5_moveit_config/config/jaka_robot.urdf.xacro (robot description, xacro)
@@ -2,8 +2,11 @@
 <robot xmlns:xacro="http://www.ros.org/wiki/xacro" name="jaka_robot">
     <xacro:arg name="initial_positions_file" default="initial_positions.yaml" />
+    <xacro:arg name="use_gazebo" default="false"/>
+    <xacro:arg name="use_rviz_sim" default="false"/>
     <!-- Import jaka_robot urdf file -->
     <xacro:include filename="$(find jaka_description)/urdf/my_robot.urdf.xacro" />
     <!-- Import control_xacro -->
     <xacro:include filename="jaka_robot.ros2_control.xacro" />
-    <xacro:jaka_robot_ros2_control name="FakeSystem" initial_positions_file="$(arg initial_positions_file)"/>
+    <!-- <xacro:jaka_robot_ros2_control name="FakeSystem" initial_positions_file="$(arg initial_positions_file)"/> -->
+     <xacro:jaka_zu5_ros2_control name="jaka_zu5_hardware" initial_positions_file="$(arg initial_positions_file)" use_gazebo="$(arg use_gazebo)" use_rviz_sim="$(arg use_rviz_sim)" />
 </robot>
