Commit message: 解决了gazebo无法使用夹爪的问题,是urdf文件最后面控制器路径设置的不对

File: jaka_description/urdf/jaka_zu5.xacro (robot description, xacro)
@@ -413,11 +413,16 @@
     <child link="tool_link" />
   </joint>
+  <!-- 定义一个传动关系，从描述关节到硬件执行器 -->
   <transmission name="trans_joint_1">
+        <!-- 线型传动关系 -->
         <type>transmission_interface/SimpleTransmission</type>
         <joint name="joint_1">
-            <hardwareInterface>hardware_interface/PositionJointInterface</hardwareInterface>
-        </joint>
+            <!-- 硬件接口为位置控制接口 -->
+            <hardwareInterface>hardware_interface/PositionJointInterface</hardwareInterface>
+        </joint>
+        <!-- 指定执行器 -->
         <actuator name="joint_1_motor">
             <hardwareInterface>hardware_interface/PositionJointInterface</hardwareInterface>
+            <!-- 定义减速比 -->
             <mechanicalReduction>1</mechanicalReduction>
         </actuator>
@@ -478,5 +483,5 @@
         <plugin name="ign_ros2_control::IgnitionROS2ControlPlugin" filename="libign_ros2_control-system.so">
           <!-- 运行 ros2_control 控制器（由 ros2_controllers.yaml 指定） -->
-          <parameters>$(find jaka_zu5_moveit_config)/config/ros2_controllers.yaml</parameters>
+          <parameters>$(find jaka_robot_moveit_config)/config/ros2_controllers.yaml</parameters>
           <robotNamespace>/</robotNamespace>
         </plugin>

File: jaka_description/urdf/my_robot.urdf.xacro (robot description, xacro)
@@ -6,11 +6,11 @@
     <!-- 如需 ros2_control，可在此包含控制描述 -->
     <!-- <xacro:include filename="my_robot.ros2_control.xacro" /> -->
-    <!-- <link name="world" /> -->
+    <link name="world" />
     <!-- 将机械臂固定在世界坐标系中 -->
-    <!-- <joint name="world_joint" type="fixed">
+    <joint name="world_joint" type="fixed">
         <parent link="world" />
         <child link="Link_0" />
         <origin xyz="0 0 0" rpy="0 0 0" />
-    </joint> -->
+    </joint>
     <!-- 将夹爪基座固定在机器人末端 tool_link 上 -->
     <joint name="gripper_base_joint" type="fixed">
