Commit message: 重命名成功

File: jaka_description/urdf/my_robot.urdf.xacro (robot description, xacro)
@@ -1,16 +1,16 @@
 <?xml version="1.0" encoding="utf-8"?>
-<robot name="jaka_robot" xmlns:xacro="http://www.ros.org/wiki/xacro">
+<robot name="jaka_zu5" xmlns:xacro="http://www.ros.org/wiki/xacro">
     <!-- 包含本包内的机器人本体与夹爪描述 -->
-    <xacro:include filename="my_jaka_zu5.xacro" />
-    <xacro:include filename="my_gripper.xacro" />
+    <xacro:include filename="jaka_zu5.xacro" />
+    <xacro:include filename="gripper.xacro" />
     <!-- 如需 ros2_control，可在此包含控制描述 -->
     <!-- <xacro:include filename="my_robot.ros2_control.xacro" /> -->
-    <link name="world" />
+    <!-- <link name="world" /> -->
     <!-- 将机械臂固定在世界坐标系中 -->
-    <joint name="world_joint" type="fixed">
+    <!-- <joint name="world_joint" type="fixed">
         <parent link="world" />
         <child link="Link_0" />
         <origin xyz="0 0 0" rpy="0 0 0" />
-    </joint>
+    </joint> -->
     <!-- 将夹爪基座固定在机器人末端 tool_link 上 -->
     <joint name="gripper_base_joint" type="fixed">

File: jaka_robot_moveit_config/config/jaka_zu5.ros2_control.xacro (robot description, xacro)
@@ -1,7 +1,8 @@
 <?xml version="1.0"?>
 <robot xmlns:xacro="http://www.ros.org/wiki/xacro">
-    <xacro:macro name="jaka_robot_ros2_control" params="name initial_positions_file use_gazebo use_rviz_sim">
+    <xacro:macro name="jaka_zu5_ros2_control" params="name initial_positions_file use_gazebo use_rviz_sim">
         <xacro:property name="initial_positions" value="${xacro.load_yaml(initial_positions_file)['initial_positions']}"/>
         <ros2_control name="${name}" type="system">
+            <!-- Include hardware plugin conditionally if rviz in simulation mode is enabled -->
             <hardware>
               <xacro:if value="${use_gazebo}">

Commit message: 准备添加相机,先保存一下

File: jaka_description/urdf/my_robot.urdf.xacro (robot description, xacro)
@@ -5,6 +5,5 @@
   <xacro:arg name="use_gazebo" default="false"/>
   <xacro:arg name="include_gripper" default="true"/>
-  <xacro:arg name="include_ros2_control" default="true"/>
-  <xacro:arg name="include_gazebo_plugins" default="false"/>
+  <xacro:arg name="include_gazebo_plugins" default="true"/>
   <!-- Include robot arm definition -->
   <xacro:include filename="$(find jaka_description)/urdf/jaka_zu5.xacro" />
@@ -12,8 +11,4 @@
   <xacro:if value="$(arg include_gripper)">
     <xacro:include filename="$(find jaka_description)/urdf/gripper.xacro" />
-  </xacro:if>
-  <!-- Include ros2_control configuration -->
-  <xacro:if value="$(arg include_ros2_control)">
-    <xacro:include filename="$(find jaka_description)/urdf/ros2_control.xacro" />
   </xacro:if>
   <!-- Include gazebo plugins and transmissions -->

File: jaka_robot_moveit_config/config/jaka_zu5.ros2_control.xacro (robot description, xacro)
@@ -1,8 +1,8 @@
 <?xml version="1.0"?>
 <robot xmlns:xacro="http://www.ros.org/wiki/xacro">
-    <xacro:macro name="jaka_zu5_ros2_control" params="name initial_positions_file use_gazebo use_rviz_sim">
+    <xacro:macro name="jaka_zu5_ros2_control" params="initial_positions_file use_gazebo use_rviz_sim">
         <xacro:property name="initial_positions" value="${xacro.load_yaml(initial_positions_file)['initial_positions']}"/>
-        <ros2_control name="${name}" type="system">
-            <!-- Include hardware plugin conditionally if rviz in simulation mode is enabled -->
+        <!-- ARM Control System - Handles joint_1 to joint_6 -->
+        <ros2_control name="jaka_arm_hardware" type="system">
             <hardware>
               <xacro:if value="${use_gazebo}">
@@ -57,4 +57,17 @@
                 <state_interface name="velocity"/>
             </joint>
+        </ros2_control>
+        <!-- Gripper Control System - Handles gripper finger joints -->
+        <ros2_control name="jaka_gripper_hardware" type="system">
+            <hardware>
+              <xacro:if value="${use_gazebo}">
+                  <plugin>gz_ros2_control/GazeboSimSystem</plugin>
+              </xacro:if>
+              <xacro:if value="${use_rviz_sim}">
+                  <plugin>fake_components/GenericSystem</plugin>
+                  <param name="mock_sensor_commands">false</param>
+                  <param name="state_following_offset">0.0</param>
+              </xacro:if>
+            </hardware>
             <joint name="gripper_left_finger_joint">
                 <command_interface name="position"/>

File: jaka_robot_moveit_config/config/jaka_zu5.urdf.xacro (robot description, xacro)
@@ -13,4 +13,4 @@
     <xacro:include filename="jaka_zu5.ros2_control.xacro" />
     <!-- Use the control macro -->
-    <xacro:jaka_zu5_ros2_control name="jaka_zu5_hardware" initial_positions_file="$(arg initial_positions_file)" use_gazebo="$(arg use_gazebo)" use_rviz_sim="$(arg use_rviz_sim)" />
+    <xacro:jaka_zu5_ros2_control initial_positions_file="$(arg initial_positions_file)" use_gazebo="$(arg use_gazebo)" use_rviz_sim="$(arg use_rviz_sim)" />
 </robot>
