Commit message: 之前一切顺利,除了右夹爪不懂,后面遇到未知原因一直启动失败,似乎是权限不够.先保存一下

File: jaka_description/urdf/gripper.xacro (robot description, xacro)
@@ -106,5 +106,4 @@
         <origin xyz="0.045 0 0.06" rpy="0 0 0" />
         <axis xyz="1 0 0" />
-        <mimic joint="gripper_left_finger_joint" multiplier="-1.0" />
         <limit effort="1000.0" velocity="1.0" lower="-0.04" upper="0.0" />
     </joint>
@@ -115,3 +114,11 @@
         <origin xyz="0 0 0.09" rpy="0 0 0" />
     </joint>
+    <ros2_control name="gripper_system" type="system">
+       <hardware>
+           <plugin>ign_ros2_control/IgnitionSystem</plugin>
+           <command_interface name="position"/>
+           <state_interface name="position"/>
+           <state_interface name="velocity"/>
+       </hardware>
+   </ros2_control>
 </robot>

File: jaka_description/urdf/jaka_zu5.xacro (robot description, xacro)
@@ -413,77 +413,105 @@
     <child link="tool_link" />
   </joint>
-  <!-- 定义一个传动关系，从描述关节到硬件执行器 -->
-  <transmission name="trans_joint_1">
-        <!-- 线型传动关系 -->
-        <type>transmission_interface/SimpleTransmission</type>
-        <joint name="joint_1">
-            <!-- 硬件接口为位置控制接口 -->
-            <hardwareInterface>hardware_interface/PositionJointInterface</hardwareInterface>
-        </joint>
-        <!-- 指定执行器 -->
-        <actuator name="joint_1_motor">
-            <hardwareInterface>hardware_interface/PositionJointInterface</hardwareInterface>
-            <!-- 定义减速比 -->
-            <mechanicalReduction>1</mechanicalReduction>
-        </actuator>
+  <ros2_control name="jaka_zu5_system" type="system">
+    <hardware>
+      <plugin>ign_ros2_control/IgnitionSystem</plugin>
+    </hardware>
+    <!-- 定义关节 -->
+    <joint name="joint_1">
+      <command_interface name="position"/>
+      <state_interface name="position"/>
+      <state_interface name="velocity"/>
+    </joint>
+    <joint name="joint_2">
+      <command_interface name="position"/>
+      <state_interface name="position"/>
+      <state_interface name="velocity"/>
+    </joint>
+    <joint name="joint_3">
+      <command_interface name="position"/>
+      <state_interface name="position"/>
+      <state_interface name="velocity"/>
+    </joint>
+    <joint name="joint_4">
+      <command_interface name="position"/>
+      <state_interface name="position"/>
+      <state_interface name="velocity"/>
+    </joint>
+    <joint name="joint_5">
+      <command_interface name="position"/>
+      <state_interface name="position"/>
+      <state_interface name="velocity"/>
+    </joint>
+    <joint name="joint_6">
+      <command_interface name="position"/>
+      <state_interface name="position"/>
+      <state_interface name="velocity"/>
+    </joint>
+    <!-- 定义传动关系：将关节映射到其物理执行器 -->
+    <transmission name="transmission_1">
+      <!-- 指定为线性传动关系 -->
+      <plugin>transmission_interface/SimpleTransmission</plugin>
+      <!-- 指定执行器 -->
+      <actuator name="joint_1_motor" role="actuator_1"/>
+      <joint name="joint_1" role="joint_1">
+        <!-- 在这里定义减速比，例如 1:1 -->
+        <mechanical_reduction>1.0</mechanical_reduction>
+        <offset>0.0</offset>
+      </joint>
     </transmission>
-    <transmission name="trans_joint_2">
-        <type>transmission_interface/SimpleTransmission</type>
-        <joint name="joint_2">
-            <hardwareInterface>hardware_interface/PositionJointInterface</hardwareInterface>
-        </joint>
-        <actuator name="joint_2_motor">
-            <hardwareInterface>hardware_interface/PositionJointInterface</hardwareInterface>
-            <mechanicalReduction>1</mechanicalReduction>
-        </actuator>
+    <transmission name="transmission_2">
+      <plugin>transmission_interface/SimpleTransmission</plugin>
+      <actuator name="joint_2_motor" role="actuator_2"/>
+      <joint name="joint_2" role="joint_2">
+        <!-- 在这里定义减速比，例如 1:1 -->
+        <mechanical_reduction>1.0</mechanical_reduction>
+        <offset>0.0</offset>
+      </joint>
     </transmission>
-    <transmission name="trans_joint_3">
-        <type>transmission_interface/SimpleTransmission</type>
-        <joint name="joint_3">
-            <hardwareInterface>hardware_interface/PositionJointInterface</hardwareInterface>
-        </joint>
-        <actuator name="joint_3_motor">
-            <hardwareInterface>hardware_interface/PositionJointInterface</hardwareInterface>
-            <mechanicalReduction>1</mechanicalReduction>
-        </actuator>
+    <transmission name="transmission_3">
+      <plugin>transmission_interface/SimpleTransmission</plugin>
+      <actuator name="joint_3_motor" role="actuator_3"/>
+      <joint name="joint_3" role="joint_3">
+        <!-- 在这里定义减速比，例如 1:1 -->
+        <mechanical_reduction>1.0</mechanical_reduction>
+        <offset>0.0</offset>
+      </joint>
     </transmission>
-    <transmission name="trans_joint_4">
-        <type>transmission_interface/SimpleTransmission</type>
-        <joint name="joint_4">
-            <hardwareInterface>hardware_interface/PositionJointInterface</hardwareInterface>
-        </joint>
-        <actuator name="joint_4_motor">
-            <hardwareInterface>hardware_interface/PositionJointInterface</hardwareInterface>
-            <mechanicalReduction>1</mechanicalReduction>
-        </actuator>
+    <transmission name="transmission_4">
+      <plugin>transmission_interface/SimpleTransmission</plugin>
+      <actuator name="joint_4_motor" role="actuator_4"/>
+      <joint name="joint_4" role="joint_4">
+        <!-- 在这里定义减速比，例如 1:1 -->
+        <mechanical_reduction>1.0</mechanical_reduction>
+        <offset>0.0</offset>
+      </joint>
     </transmission>
-    <transmission name="trans_joint_5">
-        <type>transmission_interface/SimpleTransmission</type>
-        <joint name="joint_5">
-            <hardwareInterface>hardware_interface/PositionJointInterface</hardwareInterface>
-        </joint>
-        <actuator name="joint_5_motor">
-            <hardwareInterface>hardware_interface/PositionJointInterface</hardwareInterface>
-            <mechanicalReduction>1</mechanicalReduction>
-        </actuator>
+    <transmission name="transmission_5">
+      <plugin>transmission_interface/SimpleTransmission</plugin>
+      <actuator name="joint_5_motor" role="actuator_5"/>
+      <joint name="joint_5" role="joint_5">
+        <!-- 在这里定义减速比，例如 1:1 -->
+        <mechanical_reduction>1.0</mechanical_reduction>
+        <offset>0.0</offset>
+      </joint>
     </transmission>
-    <transmission name="trans_joint_6">
-        <type>transmission_interface/SimpleTransmission</type>
-        <joint name="joint_6">
-            <hardwareInterface>hardware_interface/PositionJointInterface</hardwareInterface>
-        </joint>
-        <actuator name="joint_6_motor">
-            <hardwareInterface>hardware_interface/PositionJointInterface</hardwareInterface>
-            <mechanicalReduction>1</mechanicalReduction>
-        </actuator>
+    <transmission name="transmission_6">
+      <plugin>transmission_interface/SimpleTransmission</plugin>
+      <actuator name="joint_6_motor" role="actuator_6"/>
+      <joint name="joint_6" role="joint_6">
+        <!-- 在这里定义减速比，例如 1:1 -->
+        <mechanical_reduction>1.0</mechanical_reduction>
+        <offset>0.0</offset>
+      </joint>
     </transmission>
-    <gazebo>
-        <!-- <plugin name="gazebo_ros2_control" filename="libgazebo_ros2_control.so"> -->
-        <!--创建ros2_control 硬件接口 -->
-        <plugin name="ign_ros2_control::IgnitionROS2ControlPlugin" filename="libign_ros2_control-system.so">
-          <!-- 运行 ros2_control 控制器（由 ros2_controllers.yaml 指定） -->
-          <parameters>$(find jaka_robot_moveit_config)/config/ros2_controllers.yaml</parameters>
-          <robotNamespace>/</robotNamespace>
-        </plugin>
-    </gazebo>
+  </ros2_control>
+  <gazebo>
+      <!-- <plugin name="gazebo_ros2_control" filename="libgazebo_ros2_control.so"> -->
+      <!-- 创建 ros2_control 硬件接口（Ignition / Gazebo 仿真） -->
+      <plugin name="gz_ros2_control::GazeboSimROS2ControlPlugin" filename="libign_ros2_control-system.so">
+        <!-- 运行 ros2_control 控制器（由 ros2_controllers.yaml 指定 -->
+        <parameters>$(find jaka_robot_moveit_config)/config/ros2_controllers.yaml</parameters>
+        <robotNamespace>/</robotNamespace>
+      </plugin>
+  </gazebo>
 </robot>

File: jaka_robot_moveit_config/config/jaka_zu5.ros2_control.xacro (robot description, xacro)
@@ -7,6 +7,5 @@
             <hardware>
               <xacro:if value="${use_gazebo}">
-                  <!-- <plugin>gazebo_ros2_control/GazeboSystem</plugin> -->
-                  <plugin>ign_ros2_control/IgnitionSystem</plugin>
+                  <plugin>gz_ros2_control/IgnitionSystem</plugin>
               </xacro:if>
               <xacro:if value="${use_rviz_sim}">
@@ -63,4 +62,11 @@
                 <state_interface name="velocity"/>
             </joint>
+            <joint name="gripper_right_finger_joint">
+                <command_interface name="position"/>
+                <state_interface name="position">
+                  <param name="initial_value">${-initial_positions['gripper_left_finger_joint']}</param>
+                </state_interface>
+                <state_interface name="velocity"/>
+            </joint>
         </ros2_control>
     </xacro:macro>

Commit message: 修好了无法启动的问题,是新旧库混用导致的

File: jaka_description/urdf/gripper.xacro (robot description, xacro)
@@ -116,9 +116,16 @@
     <ros2_control name="gripper_system" type="system">
        <hardware>
-           <plugin>ign_ros2_control/IgnitionSystem</plugin>
-           <command_interface name="position"/>
-           <state_interface name="position"/>
-           <state_interface name="velocity"/>
+            <plugin>gz_ros2_control/GazeboSimSystem</plugin>
        </hardware>
+        <joint name="gripper_left_finger_joint">
+            <command_interface name="position"/>
+            <state_interface name="position"/>
+            <state_interface name="velocity"/>
+        </joint>
+        <joint name="gripper_right_finger_joint">
+            <command_interface name="position"/>
+            <state_interface name="position"/>
+            <state_interface name="velocity"/>
+        </joint>
    </ros2_control>
 </robot>

File: jaka_description/urdf/jaka_zu5.xacro (robot description, xacro)
@@ -415,5 +415,5 @@
   <ros2_control name="jaka_zu5_system" type="system">
     <hardware>
-      <plugin>ign_ros2_control/IgnitionSystem</plugin>
+      <plugin>gz_ros2_control/GazeboSimSystem</plugin>
     </hardware>
     <!-- 定义关节 -->

Commit message: 现在only rviz 和 rviz+gazebo 都运行正常,是使用控制插件不对导致的,rviz的假仿真需要假插件

File: jaka_description/urdf/gripper.xacro (robot description, xacro)
@@ -1,4 +1,4 @@
 <?xml version="1.0" encoding="utf-8"?>
-<robot xmlns:xacro="http://www.ros.org/wiki/xacro">
+<robot name="jaka_gripper" xmlns:xacro="http://www.ros.org/wiki/xacro">
     <material name="dark_green">
         <color rgba="0 0.4 0 1" />
@@ -86,12 +86,12 @@
     </link>
     <!-- 抓取点的位置，用虚拟连杆占位 -->
-    <link name="grip_center_link">
+    <!-- <link name="grip_center_link"> -->
         <!-- 没有视觉和碰撞，只有惯性属性 -->
-        <inertial>
+        <!-- <inertial>
             <origin xyz="0 0 0" rpy="0 0 0" />
             <mass value="0.0001" />
             <inertia ixx="1e-06" ixy="0" ixz="0" iyy="1e-06" iyz="0" izz="1e-06" />
         </inertial>
-    </link>
+    </link> -->
     <joint name="gripper_left_finger_joint" type="prismatic">
         <parent link="gripper_base_link" />
@@ -109,23 +109,14 @@
     </joint>
     <!-- 抓取点 -->
-    <joint name="grip_center_joint" type="fixed">
+    <!-- <joint name="grip_center_joint" type="fixed">
         <parent link="gripper_base_link" />
         <child link="grip_center_link" />
         <origin xyz="0 0 0.09" rpy="0 0 0" />
+    </joint> -->
+  <!-- Joint to connect gripper to robot arm -->
+    <joint name="gripper_joint" type="fixed">
+        <parent link="tool_link" />
+        <child link="gripper_base_link" />
+        <origin xyz="0 0 0" rpy="0 0 0" />
     </joint>
-    <ros2_control name="gripper_system" type="system">
-       <hardware>
-            <plugin>gz_ros2_control/GazeboSimSystem</plugin>
-       </hardware>
-        <joint name="gripper_left_finger_joint">
-            <command_interface name="position"/>
-            <state_interface name="position"/>
-            <state_interface name="velocity"/>
-        </joint>
-        <joint name="gripper_right_finger_joint">
-            <command_interface name="position"/>
-            <state_interface name="position"/>
-            <state_interface name="velocity"/>
-        </joint>
-   </ros2_control>
 </robot>

File: jaka_description/urdf/jaka_zu5.xacro (robot description, xacro)
@@ -3,5 +3,5 @@
      Commit Version: 1.5.1-0-g916b5db  Build Version: 1.5.7152.31018
      For more information, please see http://wiki.ros.org/sw_urdf_exporter -->
-<robot xmlns:xacro="http://www.ros.org/wiki/xacro">
+<robot name="jaka_zu5_arm" xmlns:xacro="http://www.ros.org/wiki/xacro">
   <!-- LINK -->
   <!-- <link name="base_link" /> -->
@@ -413,105 +413,3 @@
     <child link="tool_link" />
   </joint>
-  <ros2_control name="jaka_zu5_system" type="system">
-    <hardware>
-      <plugin>gz_ros2_control/GazeboSimSystem</plugin>
-    </hardware>
-    <!-- 定义关节 -->
-    <joint name="joint_1">
-      <command_interface name="position"/>
-      <state_interface name="position"/>
-      <state_interface name="velocity"/>
-    </joint>
-    <joint name="joint_2">
-      <command_interface name="position"/>
-      <state_interface name="position"/>
-      <state_interface name="velocity"/>
-    </joint>
-    <joint name="joint_3">
-      <command_interface name="position"/>
-      <state_interface name="position"/>
-      <state_interface name="velocity"/>
-    </joint>
-    <joint name="joint_4">
-      <command_interface name="position"/>
-      <state_interface name="position"/>
-      <state_interface name="velocity"/>
-    </joint>
-    <joint name="joint_5">
-      <command_interface name="position"/>
-      <state_interface name="position"/>
-      <state_interface name="velocity"/>
-    </joint>
-    <joint name="joint_6">
-      <command_interface name="position"/>
-      <state_interface name="position"/>
-      <state_interface name="velocity"/>
-    </joint>
-    <!-- 定义传动关系：将关节映射到其物理执行器 -->
-    <transmission name="transmission_1">
-      <!-- 指定为线性传动关系 -->
-      <plugin>transmission_interface/SimpleTransmission</plugin>
-      <!-- 指定执行器 -->
-      <actuator name="joint_1_motor" role="actuator_1"/>
-      <joint name="joint_1" role="joint_1">
-        <!-- 在这里定义减速比，例如 1:1 -->
-        <mechanical_reduction>1.0</mechanical_reduction>
-        <offset>0.0</offset>
-      </joint>
-    </transmission>
-    <transmission name="transmission_2">
-      <plugin>transmission_interface/SimpleTransmission</plugin>
-      <actuator name="joint_2_motor" role="actuator_2"/>
-      <joint name="joint_2" role="joint_2">
-        <!-- 在这里定义减速比，例如 1:1 -->
-        <mechanical_reduction>1.0</mechanical_reduction>
-        <offset>0.0</offset>
-      </joint>
-    </transmission>
-    <transmission name="transmission_3">
-      <plugin>transmission_interface/SimpleTransmission</plugin>
-      <actuator name="joint_3_motor" role="actuator_3"/>
-      <joint name="joint_3" role="joint_3">
-        <!-- 在这里定义减速比，例如 1:1 -->
-        <mechanical_reduction>1.0</mechanical_reduction>
-        <offset>0.0</offset>
-      </joint>
-    </transmission>
-    <transmission name="transmission_4">
-      <plugin>transmission_interface/SimpleTransmission</plugin>
-      <actuator name="joint_4_motor" role="actuator_4"/>
-      <joint name="joint_4" role="joint_4">
-        <!-- 在这里定义减速比，例如 1:1 -->
-        <mechanical_reduction>1.0</mechanical_reduction>
-        <offset>0.0</offset>
-      </joint>
-    </transmission>
-    <transmission name="transmission_5">
-      <plugin>transmission_interface/SimpleTransmission</plugin>
-      <actuator name="joint_5_motor" role="actuator_5"/>
-      <joint name="joint_5" role="joint_5">
-        <!-- 在这里定义减速比，例如 1:1 -->
-        <mechanical_reduction>1.0</mechanical_reduction>
-        <offset>0.0</offset>
-      </joint>
-    </transmission>
-    <transmission name="transmission_6">
-      <plugin>transmission_interface/SimpleTransmission</plugin>
-      <actuator name="joint_6_motor" role="actuator_6"/>
-      <joint name="joint_6" role="joint_6">
-        <!-- 在这里定义减速比，例如 1:1 -->
-        <mechanical_reduction>1.0</mechanical_reduction>
-        <offset>0.0</offset>
-      </joint>
-    </transmission>
-  </ros2_control>
-  <gazebo>
-      <!-- <plugin name="gazebo_ros2_control" filename="libgazebo_ros2_control.so"> -->
-      <!-- 创建 ros2_control 硬件接口（Ignition / Gazebo 仿真） -->
-      <plugin name="gz_ros2_control::GazeboSimROS2ControlPlugin" filename="libign_ros2_control-system.so">
-        <!-- 运行 ros2_control 控制器（由 ros2_controllers.yaml 指定 -->
-        <parameters>$(find jaka_robot_moveit_config)/config/ros2_controllers.yaml</parameters>
-        <robotNamespace>/</robotNamespace>
-      </plugin>
-  </gazebo>
 </robot>

File: jaka_description/urdf/my_robot.urdf.xacro (robot description, xacro)
@@ -1,21 +1,31 @@
 <?xml version="1.0" encoding="utf-8"?>
+<!-- Main robot URDF file that combines all robot components -->
 <robot name="jaka_zu5" xmlns:xacro="http://www.ros.org/wiki/xacro">
-    <!-- 包含本包内的机器人本体与夹爪描述 -->
-    <xacro:include filename="jaka_zu5.xacro" />
-    <xacro:include filename="gripper.xacro" />
-    <!-- 如需 ros2_control，可在此包含控制描述 -->
-    <!-- <xacro:include filename="my_robot.ros2_control.xacro" /> -->
-    <link name="world" />
-    <!-- 将机械臂固定在世界坐标系中 -->
-    <joint name="world_joint" type="fixed">
-        <parent link="world" />
-        <child link="Link_0" />
-        <origin xyz="0 0 0" rpy="0 0 0" />
-    </joint>
-    <!-- 将夹爪基座固定在机器人末端 tool_link 上 -->
-    <joint name="gripper_base_joint" type="fixed">
-        <parent link="tool_link" />
-        <child link="gripper_base_link" />
-        <origin xyz="0 0 0" rpy="0 0 0" />
-    </joint>
+  <!-- Define arguments for configuration -->
+  <xacro:arg name="use_gazebo" default="false"/>
+  <xacro:arg name="include_gripper" default="true"/>
+  <xacro:arg name="include_ros2_control" default="true"/>
+  <xacro:arg name="include_gazebo_plugins" default="false"/>
+  <!-- Include robot arm definition -->
+  <xacro:include filename="$(find jaka_description)/urdf/jaka_zu5.xacro" />
+  <!-- Include gripper definition if needed -->
+  <xacro:if value="$(arg include_gripper)">
+    <xacro:include filename="$(find jaka_description)/urdf/gripper.xacro" />
+  </xacro:if>
+  <!-- Include ros2_control configuration -->
+  <xacro:if value="$(arg include_ros2_control)">
+    <xacro:include filename="$(find jaka_description)/urdf/ros2_control.xacro" />
+  </xacro:if>
+  <!-- Include gazebo plugins and transmissions -->
+  <xacro:if value="$(arg include_gazebo_plugins)">
+    <xacro:include filename="$(find jaka_description)/urdf/gazebo.xacro" />
+  </xacro:if>
+  <!-- World link for ground truth -->
+  <link name="world" />
+  <!-- Fix robot arm to world coordinate system -->
+  <joint name="world_joint" type="fixed">
+    <parent link="world" />
+    <child link="Link_0" />
+    <origin xyz="0 0 0" rpy="0 0 0" />
+  </joint>
 </robot>

File: jaka_robot_moveit_config/config/jaka_zu5.ros2_control.xacro (robot description, xacro)
@@ -7,8 +7,10 @@
             <hardware>
               <xacro:if value="${use_gazebo}">
-                  <plugin>gz_ros2_control/IgnitionSystem</plugin>
+                  <plugin>gz_ros2_control/GazeboSimSystem</plugin>
               </xacro:if>
               <xacro:if value="${use_rviz_sim}">
-                  <plugin>mock_components/GenericSystem</plugin>
+                  <plugin>fake_components/GenericSystem</plugin>
+                  <param name="mock_sensor_commands">false</param>
+                  <param name="state_following_offset">0.0</param>
               </xacro:if>
             </hardware>

File: jaka_robot_moveit_config/config/jaka_zu5.urdf.xacro (robot description, xacro)
@@ -4,9 +4,13 @@
     <xacro:arg name="use_gazebo" default="false"/>
     <xacro:arg name="use_rviz_sim" default="true"/>
+    <!-- Arguments to pass to my_robot.urdf.xacro -->
+    <xacro:arg name="include_gripper" default="true"/>
+    <xacro:arg name="include_ros2_control" default="false"/>  <!-- We'll use the control from jaka_zu5.ros2_control.xacro -->
+    <xacro:arg name="include_gazebo_plugins" default="$(arg use_gazebo)"/>
     <!-- Import jaka_zu5 urdf file -->
     <xacro:include filename="$(find jaka_description)/urdf/my_robot.urdf.xacro" />
     <!-- Import control_xacro -->
     <xacro:include filename="jaka_zu5.ros2_control.xacro" />
-    <!-- <xacro:jaka_zu5_ros2_control name="FakeSystem" initial_positions_file="$(arg initial_positions_file)"/> -->
+    <!-- Use the control macro -->
     <xacro:jaka_zu5_ros2_control name="jaka_zu5_hardware" initial_positions_file="$(arg initial_positions_file)" use_gazebo="$(arg use_gazebo)" use_rviz_sim="$(arg use_rviz_sim)" />
 </robot>

Commit message: 成功将相机模型添加到机械臂上,即将获取图像信息

File: jaka_description/urdf/gripper.xacro (robot description, xacro)
@@ -115,5 +115,5 @@
     </joint> -->
   <!-- Joint to connect gripper to robot arm -->
-    <joint name="gripper_joint" type="fixed">
+    <joint name="gripper_base_joint" type="fixed">
         <parent link="tool_link" />
         <child link="gripper_base_link" />

File: jaka_description/urdf/my_robot.urdf.xacro (robot description, xacro)
@@ -6,4 +6,5 @@
   <xacro:arg name="include_gripper" default="true"/>
   <xacro:arg name="include_gazebo_plugins" default="true"/>
+  <xacro:property name="PI" value="3.14159274"/>
   <!-- Include robot arm definition -->
   <xacro:include filename="$(find jaka_description)/urdf/jaka_zu5.xacro" />
@@ -12,4 +13,10 @@
     <xacro:include filename="$(find jaka_description)/urdf/gripper.xacro" />
   </xacro:if>
+  <!-- 添加相机 -->
+  <xacro:include filename="$(find jaka_description)/urdf/camera.xacro" />
+  <xacro:camera_v0 parent="gripper_base_link">
+        <origin xyz="0 -0.06 0.03" rpy="${-PI/2} ${-PI/2} 0"/>
+  </xacro:camera_v0>
+  <xacro:camera_gazebo_v0/>
   <!-- Include gazebo plugins and transmissions -->
   <xacro:if value="$(arg include_gazebo_plugins)">
