Commit message: 目前已实现了图像信息的桥接转发到了ros2中,但是还没有可视化成功

File: jaka_description/urdf/camera.xacro (robot description, xacro)
@@ -20,5 +20,5 @@
 			<collision>
 				<geometry>
-					<mesh filename="package://jaka_description/meshes/camera/camera.stl"/>
+					<mesh filename="packa ge://jaka_description/meshes/camera/camera.stl"/>
 				</geometry>
 			</collision>

File: jaka_description/urdf/my_robot.urdf.xacro (robot description, xacro)
@@ -2,25 +2,11 @@
 <!-- Main robot URDF file that combines all robot components -->
 <robot name="jaka_zu5" xmlns:xacro="http://www.ros.org/wiki/xacro">
-  <!-- Define arguments for configuration -->
-  <xacro:arg name="use_gazebo" default="false"/>
-  <xacro:arg name="include_gripper" default="true"/>
-  <xacro:arg name="include_gazebo_plugins" default="true"/>
   <xacro:property name="PI" value="3.14159274"/>
   <!-- Include robot arm definition -->
   <xacro:include filename="$(find jaka_description)/urdf/jaka_zu5.xacro" />
   <!-- Include gripper definition if needed -->
-  <xacro:if value="$(arg include_gripper)">
-    <xacro:include filename="$(find jaka_description)/urdf/gripper.xacro" />
-  </xacro:if>
-  <!-- 添加相机 -->
-  <xacro:include filename="$(find jaka_description)/urdf/camera.xacro" />
-  <xacro:camera_v0 parent="gripper_base_link">
-        <origin xyz="0 -0.06 0.03" rpy="${-PI/2} ${-PI/2} 0"/>
-  </xacro:camera_v0>
-  <xacro:camera_gazebo_v0/>
-  <!-- Include gazebo plugins and transmissions -->
-  <xacro:if value="$(arg include_gazebo_plugins)">
-    <xacro:include filename="$(find jaka_description)/urdf/gazebo.xacro" />
-  </xacro:if>
+  <xacro:include filename="$(find jaka_description)/urdf/gripper.xacro" />
+  <!-- 添加传动配置 -->
+  <xacro:include filename="$(find jaka_description)/urdf/jaka_zu5.gazebo" />
   <!-- World link for ground truth -->
   <link name="world" />

File: jaka_robot_moveit_config/config/jaka_zu5.urdf.xacro (robot description, xacro)
@@ -5,9 +5,18 @@
     <xacro:arg name="use_rviz_sim" default="true"/>
     <!-- Arguments to pass to my_robot.urdf.xacro -->
-    <xacro:arg name="include_gripper" default="true"/>
-    <xacro:arg name="include_ros2_control" default="false"/>  <!-- We'll use the control from jaka_zu5.ros2_control.xacro -->
-    <xacro:arg name="include_gazebo_plugins" default="$(arg use_gazebo)"/>
+    <!-- <xacro:arg name="include_ros2_control" default="false"/>  We'll use the control from jaka_zu5.ros2_control.xacro -->
     <!-- Import jaka_zu5 urdf file -->
     <xacro:include filename="$(find jaka_description)/urdf/my_robot.urdf.xacro" />
+      <!-- 添加相机 -->
+  <xacro:include filename="$(find jaka_description)/urdf/camera.xacro" />
+  <xacro:camera_v0 parent="gripper_base_link">
+        <origin xyz="0 -0.06 0.03" rpy="${-PI/2} ${-PI/2} 0"/>
+  </xacro:camera_v0>
+  <xacro:camera_gazebo_v0/>
+  <gazebo>
+        <plugin filename="ignition-gazebo-sensors-system" name="ignition::gazebo::systems::Sensors">
+            <!-- <render_engine>ogre2</render_engine> -->
+        </plugin>
+    </gazebo>
     <!-- Import control_xacro -->
     <xacro:include filename="jaka_zu5.ros2_control.xacro" />
